Commit message: Update

File: description/robot.urdf.xacro (robot description, xacro)
@@ -3,3 +3,4 @@
     <!-- Example link -->
     <xacro:include filename="robot_core.xacro"/>
+    <xacro:include filename="gazebo_control.xacro"/>
 </robot>

File: description/robot_core.xacro (robot description, xacro)
@@ -41,4 +41,7 @@
         </xacro:inertial_box>
     </link>
+<gazebo reference="chassis">
+<material>Gazebo/Blue</material>
+</gazebo>
 <!-- Left Wheel Link-->
     <joint name="left_wheel_joint" type="continuous">
@@ -64,4 +67,7 @@
         </xacro:inertial_cylinder>
     </link>
+<gazebo reference="left_wheel">
+<material>Gazebo/Black</material>
+</gazebo>
 <!-- Right Wheel Link-->
     <joint name="right_wheel_joint" type="continuous">
@@ -87,4 +93,7 @@
         </xacro:inertial_cylinder>
     </link>
+    <gazebo reference="right_wheel">
+<material>Gazebo/Black</material>
+</gazebo>
 <!-- Caster Wheel Link-->
     <joint name="caster_wheel_joint" type="fixed">
@@ -109,3 +118,8 @@
         </xacro:inertial_sphere>
     </link>
+        <gazebo reference="caster_wheel">
+<material>Gazebo/Black</material>
+<mu1 value="0.0001"/>
+<mu2 value="0.0001"/>
+</gazebo>
 </robot>
